File: kicad/ehz-diag.sch (KiCad schematic (older format))
At the start: 14 parts, among them J1 Screw-Terminal, Q1 SFH309FA, Q2 BC557, Q3 BC548

Commit message: Issue #1: Schaltplan Rev. 1.1
- J1: Farben in Beschriftung korrigiert
- R2: Beschriftung gedreht
Other:
- note added: "Beschriftung:\nC: Collector / Pin 4 / weiß\nA: Anode / Pin 3 / gelb\nK: Kathode / Pin 2 / grün\nE: Emitter / Pin 1 / braun\n\n"
- note removed: "Beschriftung:\nC: Collector / Pin 4 / braun\nA: Anode / Pin 3 / gelb\nK: Kathode / Pin 2 / grün\nE: Emitter / Pin 1 / weiß\n\n"
Changed lines of the file:
@@
 Sheet 1 1
 Title "EHZ Diagnose-Tool 1-Kanal mit Buzzer"
-Date "2021-08-29"
-Rev "1.0"
+Date "2021-09-05"
+Rev "1.1"
 Comp "Andreas Dolp"
 Comment1 "GitHub: e-cite/ehz-diag"
@@
 $EndComp
 Text Notes 3150 3800 0    50   ~ 0
-Beschriftung:\nC: Collector / Pin 4 / braun\nA: Anode / Pin 3 / gelb\nK: Kathode / Pin 2 / grün\nE: Emitter / Pin 1 / weiß\n\n
+Beschriftung:\nC: Collector / Pin 4 / weiß\nA: Anode / Pin 3 / gelb\nK: Kathode / Pin 2 / grün\nE: Emitter / Pin 1 / braun\n\n
 $Comp
 L Device:R R4
@@
 U 1 1 6129C2D2
 P 6900 3300
-F 0 "R2" V 7100 3300 50  0000 C CNN
-F 1 "10k" V 7000 3300 50  0000 C CNN
+F 0 "R2" H 7000 3350 50  0000 L CNN
+F 1 "10k" H 7000 3250 50  0000 L CNN
 F 2 "Resistor_THT:R_Axial_DIN0207_L6.3mm_D2.5mm_P15.24mm_Horizontal" V 6830 3300 50  0001 C CNN
 F 3 "~" H 6900 3300 50  0001 C CNN
